File: IO.sch (KiCad schematic (older format))
At the start: 27 parts, among them J6 OUT, J7 I2C, Q1 2N7002, Q2 BC817, Q3 DNP, Q4 DNP, Q5 DNP, Q6 DNP, U13 USBLC6-4, U8 DRV8837

Commit message: exported gerbers
Parts:
- C21, C23: value 100n -> DNP
- C22: value 1uF -> DNP
- Q3, Q5: value DNP -> 2N7002
- Q4, Q6: value DNP -> BC817
- R20, R21, R22, R23: value DNP -> 220
Connections:
- net SCL: now also J7.3 (Pin_3), R17.1, U13.3 (IO2); no longer J7.2 (Pin_2), R16.2, U13.1 (IO1)
- net SDA: now also J7.2 (Pin_2), R16.2, U13.1 (IO1); no longer J7.3 (Pin_3), R17.1, U13.3 (IO2)
Changed lines of the file:
@@
 AR Path="/6188CC74/61891D60" Ref="C23"  Part="1"
 F 0 "C23" H 6908 1404 50  0000 R CNN
-F 1 "100n" H 6908 1495 50  0000 R CNN
+F 1 "DNP" H 6908 1495 50  0000 R CNN
 F 2 "otter:C_0402" H 7000 1450 50  0001 C CNN
 F 3 "~" H 7000 1450 50  0001 C CNN
@@
 AR Path="/6188CC74/61891D72" Ref="C22"  Part="1"
 F 0 "C22" H 5958 1254 50  0000 R CNN
-F 1 "1uF" H 5958 1345 50  0000 R CNN
+F 1 "DNP" H 5958 1345 50  0000 R CNN
 F 2 "otter:C_0603" H 6050 1300 50  0001 C CNN
 F 3 "~" H 6050 1300 50  0001 C CNN
@@
 AR Path="/6188CC74/61891D7E" Ref="C21"  Part="1"
 F 0 "C21" H 5608 1254 50  0000 R CNN
-F 1 "100n" H 5608 1345 50  0000 R CNN
+F 1 "DNP" H 5608 1345 50  0000 R CNN
 F 2 "otter:C_0402" H 5700 1300 50  0001 C CNN
 F 3 "~" H 5700 1300 50  0001 C CNN
@@
 AR Path="/6188CC74/618A4D42" Ref="Q3"  Part="1"
 F 0 "Q3" H 3755 2546 50  0000 L CNN
-F 1 "DNP" H 3755 2455 50  0000 L CNN
+F 1 "2N7002" H 3755 2455 50  0000 L CNN
 F 2 "Package_TO_SOT_SMD:SOT-23" H 3750 2425 50  0001 L CIN
 F 3 "https://www.fairchildsemi.com/datasheets/2N/2N7002.pdf" H 3550 2500 50  0001 L CNN
@@
 AR Path="/6188CC74/618A4D4F" Ref="Q4"  Part="1"
 F 0 "Q4" H 4191 2746 50  0000 L CNN
-F 1 "DNP" H 4191 2655 50  0000 L CNN
+F 1 "BC817" H 4191 2655 50  0000 L CNN
 F 2 "Package_TO_SOT_SMD:SOT-23" H 4200 2625 50  0001 L CIN
 F 3 "http://www.fairchildsemi.com/ds/BC/BC817.pdf" H 4000 2700 50  0001 L CNN
@@
 AR Path="/6188CC74/618A4D5D" Ref="R21"  Part="1"
 F 0 "R21" V 4496 2700 50  0000 C CNN
-F 1 "DNP" V 4405 2700 50  0000 C CNN
+F 1 "220" V 4405 2700 50  0000 C CNN
 F 2 "otter:R_0402" H 4300 2700 50  0001 C CNN
 F 3 "~" H 4300 2700 50  0001 C CNN
@@
 AR Path="/6188CC74/618A4D63" Ref="R20"  Part="1"
 F 0 "R20" H 3741 2304 50  0000 R CNN
-F 1 "DNP" H 3741 2395 50  0000 R CNN
+F 1 "220" H 3741 2395 50  0000 R CNN
 F 2 "otter:R_0402" H 3800 2350 50  0001 C CNN
 F 3 "~" H 3800 2350 50  0001 C CNN
@@
 Wire Wire Line
 	3800 2500 3750 2500
-$Comp
-L Transistor_FET:2N7002 Q?
-U 1 1 618A8469
-P 4950 2500
-AR Path="/618A8469" Ref="Q?"  Part="1"
-AR Path="/6188CC74/618A8469" Ref="Q5"  Part="1"
-F 0 "Q5" H 5155 2546 50  0000 L CNN
-F 1 "DNP" H 5155 2455 50  0000 L CNN
-F 2 "Package_TO_SOT_SMD:SOT-23" H 5150 2425 50  0001 L CIN
-F 3 "https://www.fairchildsemi.com/datasheets/2N/2N7002.pdf" H 4950 2500 50  0001 L CNN
-	1    4950 2500
-	-1   0    0    -1
-$EndComp
 $Comp
 L otter:GND #PWR?
@@
 AR Path="/6188CC74/618A8476" Ref="Q6"  Part="1"
 F 0 "Q6" H 5591 2746 50  0000 L CNN
-F 1 "DNP" H 5591 2655 50  0000 L CNN
+F 1 "BC817" H 5591 2655 50  0000 L CNN
 F 2 "Package_TO_SOT_SMD:SOT-23" H 5600 2625 50  0001 L CIN
 F 3 "http://www.fairchildsemi.com/ds/BC/BC817.pdf" H 5400 2700 50  0001 L CNN
@@
 AR Path="/6188CC74/618A8484" Ref="R23"  Part="1"
 F 0 "R23" V 5896 2700 50  0000 C CNN
-F 1 "DNP" V 5805 2700 50  0000 C CNN
+F 1 "220" V 5805 2700 50  0000 C CNN
 F 2 "otter:R_0402" H 5700 2700 50  0001 C CNN
 F 3 "~" H 5700 2700 50  0001 C CNN
@@
 AR Path="/6188CC74/618A848A" Ref="R22"  Part="1"
 F 0 "R22" H 5141 2304 50  0000 R CNN
-F 1 "DNP" H 5141 2395 50  0000 R CNN
+F 1 "220" H 5141 2395 50  0000 R CNN
 F 2 "otter:R_0402" H 5200 2350 50  0001 C CNN
 F 3 "~" H 5200 2350 50  0001 C CNN
@@
 Wire Wire Line
 	5200 1900 5200 2250
+Text HLabel 1950 4250 2    50   Input ~ 0
+SDA
 Text HLabel 1950 4150 2    50   Input ~ 0
-SDA
-Text HLabel 1950 4250 2    50   Input ~ 0
 SCL
 Text HLabel 3000 2700 2    50   Input ~ 0
@@
 Wire Wire Line
 	3450 2100 5900 2100
+$Comp
+L Transistor_FET:2N7002 Q?
+U 1 1 618A8469
+P 4950 2500
+AR Path="/618A8469" Ref="Q?"  Part="1"
+AR Path="/6188CC74/618A8469" Ref="Q5"  Part="1"
+F 0 "Q5" H 5155 2546 50  0000 L CNN
+F 1 "2N7002" H 5155 2455 50  0000 L CNN
+F 2 "Package_TO_SOT_SMD:SOT-23" H 5150 2425 50  0001 L CIN
+F 3 "https://www.fairchildsemi.com/datasheets/2N/2N7002.pdf" H 4950 2500 50  0001 L CNN
+	1    4950 2500
+	-1   0    0    -1
+$EndComp
 $EndSCHEMATC
