File: temperature-logger.kicad_pcb (KiCad board)
At the start: 4 copper layers, 106 x 50 mm, 155 parts, among them J1 USB, J10 DNP, J11 DNP, J2 THERMOCOUPLE, J3 THERMOCOUPLE, J4 THERMOCOUPLE, J5 THERMOCOUPLE, J6 OUT, J7 I2C, J8 DNP, J9 DNP, P1 TC2030, Q1 2N7002, Q2 BC817, Q3 DNP, Q4 DNP, Q5 DNP, Q6 DNP, SW1 SCPI_CSV, U1 USBLC6-4, U10 TLV9001, U11 TLV9001, U12 TLV9001, U13 USBLC6-4, U2 AP2204R-3.3, U3 STM32F072C8Tx, U4 MAX31855KASA, U5 MAX31855KASA, U6 MAX31855KASA, U7 MAX31855KASA, U8 DRV8837, U9 TLV9001

Commit message: exported gerbers
Parts:
- added G***: LOGO, otter:usb-temperature-logger-back-text, B.Cu at (90.6, 70.0)
- added G***: LOGO, otter:usb-temperature-logger-front-text, F.Cu at (79.1, 67.4)
- moved C24 0.27 mm to (126.7, 59.3)
Connections:
- J7 pad 2: SCL -> SDA
- J7 pad 3: SDA -> SCL
- R16 pad 2: SCL -> SDA
- R17 pad 1: SDA -> SCL
- U13 pad 1: SCL -> SDA
- U13 pad 3: SDA -> SCL
Routing:
- net +3V3: track 125.3 -> 399.7 mm, vias 1 -> 20
- net NTC3: track 8.31 -> 70.4 mm, vias 0 -> 2
- net CS3: track 0.00 -> 56.3 mm, vias 0 -> 2
- net SCL: track 5.36 -> 56.3 mm
- net NTC2: track 8.29 -> 54.8 mm, vias 0 -> 2
- net SDA: track 5.24 -> 51.4 mm
- net OUT_nSLEEP: track 0.00 -> 39.2 mm, vias 0 -> 2
- net NTC_BOARD: track 1.64 -> 35.7 mm, vias 0 -> 2
- net CS2: track 0.00 -> 31.0 mm, vias 0 -> 2
- net NTC1: track 8.21 -> 35.5 mm, vias 0 -> 2
- net GND: track 19.3 -> 42.6 mm, vias 4 -> 197
- net Net-(FB7-Pad1): track 17.9 -> 40.5 mm, vias 0 -> 1
- net STATUS_LED: track 1.52 -> 21.5 mm
- net Net-(FB1-Pad1): track 17.9 -> 35.7 mm, vias 0 -> 1
- net Net-(FB3-Pad1): track 17.9 -> 35.7 mm, vias 0 -> 1
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- added copper zone on B.Cu, net GND
- added copper zone on F.Cu, net GND
- added copper zone on In1.Cu, net GND
- added copper zone on In2.Cu, net GND
Other:
- board text added: "3V3"
- board text added: "CSV - SCPI"
- board text added: "DFU"
- board text added: "GND"
- board text added: "IN0"
- board text added: "IN1"
- board text added: "IN2"
- board text added: "IN3"
- board text added: "OUT0"
- board text added: "OUT1"
- board text added: "OUT2"
- board text added: "SCL"
- board text added: "SDA"
- board text added: "VBUS"
- board text added: "VM"
