File: temperature-logger.kicad_pcb (KiCad board)
At the start: 4 copper layers, 106 x 50 mm, 157 parts, among them J1 USB, J10 DNP, J11 DNP, J2 THERMOCOUPLE, J3 THERMOCOUPLE, J4 THERMOCOUPLE, J5 THERMOCOUPLE, J6 OUT, J7 I2C, J8 DNP, J9 DNP, P1 TC2030, Q1 2N7002, Q2 BC817, Q3 DNP, Q4 DNP, Q5 DNP, Q6 DNP, SW1 SCPI_CSV, U1 USBLC6-4, U10 TLV9001, U11 TLV9001, U12 TLV9001, U13 USBLC6-4, U2 AP2204R-3.3, U3 STM32F072C8Tx, U4 MAX31855KASA, U5 MAX31855KASA, U6 MAX31855KASA, U7 MAX31855KASA, U8 DRV8837, U9 TLV9001

Commit message: updated to kicad 6
Other:
- net class Default removed

Commit message: fixed isses #1
Parts:
- C21, C23: value 100n -> DNP
- C22: value 1uF -> DNP
- Q3, Q5: value DNP -> 2N7002
- Q4, Q6: value DNP -> BC817
- R20, R21, R22, R23: value DNP -> 220
- R27, R28: value 220 -> 5k1
- moved C24 7.31 mm to (127.0, 66.6)
Connections:
- J1 pad A8: Net-(J1-PadA8) -> unconnected-(J1-PadA8)
- J1 pad B8: Net-(J1-PadB8) -> unconnected-(J1-PadB8)
- P1 pad 3: Net-(P1-Pad3) -> unconnected-(P1-Pad3)
- P1 pad 6: Net-(P1-Pad6) -> unconnected-(P1-Pad6)
- U1 pad 1: Net-(U1-Pad1) -> unconnected-(U1-Pad1)
- U1 pad 3: Net-(U1-Pad3) -> unconnected-(U1-Pad3)
- U13 pad 4: Net-(U13-Pad4) -> unconnected-(U13-Pad4)
- U13 pad 6: Net-(U13-Pad6) -> unconnected-(U13-Pad6)
- U3 pad 18: Net-(U3-Pad18) -> NTC_BOARD
- U3 pad 19: Net-(U3-Pad19) -> unconnected-(U3-Pad19)
- U3 pad 20: Net-(U3-Pad20) -> unconnected-(U3-Pad20)
- U3 pad 21: Net-(U3-Pad21) -> unconnected-(U3-Pad21)
- U3 pad 22: Net-(U3-Pad22) -> unconnected-(U3-Pad22)
- U3 pad 25: Net-(U3-Pad25) -> unconnected-(U3-Pad25)
- U3 pad 26: Net-(U3-Pad26) -> unconnected-(U3-Pad26)
- U3 pad 27: Net-(U3-Pad27) -> unconnected-(U3-Pad27)
- U3 pad 28: Net-(U3-Pad28) -> unconnected-(U3-Pad28)
- U3 pad 29: NTC_BOARD -> unconnected-(U3-Pad29)
- U3 pad 6: Net-(U3-Pad6) -> unconnected-(U3-Pad6)
Routing:
- net Net-(JP1-Pad1): track 16.6 -> 12.7 mm, vias 2 -> 1
- net NTC_BOARD: track 35.7 -> 34.3 mm
- net GND: track 42.6 -> 43.2 mm, vias 197 -> 199
- net +3V3: track 399.7 -> 400.0 mm, vias 20 -> 19
