File: temperature-logger.sch (KiCad schematic (older format))
At the start: 36 parts, among them J1 USB, P1 TC2030, SW1 SCPI_CSV, U1 USBLC6-4, U2 AP2204R-3.3, U3 STM32F072C8Tx

Commit message: exported gerbers
Parts:
- R27, R28: value 220 -> 5k1
Other:
- note removed: "Temperatur logger bauen\nZwei gestackte bords, eins nur als Blende\nRoter 3D Druck dazwischen\nMit locator holes DONE\nOpen collector Ausgänge DONE\nUSB cdc + Scpi DONE\nOnboard ref sensor gut Isolieren DONE\n4 temp inputs DONE\nOtter vorne drauf mit temperaturmessung an Nase \nTag connect hinten DONE\nLED für Status DONE\nNTC inputs? DONE\nI2C Exposed DONE\nAlternate 3.5mm input temperature DONE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"
- moved on the sheet: C10, C11, C6, C7, D10, D11, D9, H1, H2, H3, H4, J1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
