File: tsens.sch (KiCad schematic (older format))
At the start: 23 parts, among them J2 THERMOCOUPLE, J8 DNP, U4 MAX31855KASA, U9 TLV9001

Commit message: exported gerbers
Parts:
- gave numbers to parts that had none: 1
Other:
- moved on the sheet: R34
Changed lines of the file:
@@
 Connection ~ 5750 2000
-Wire Wire Line
-	5750 2000 6000 2000
 Wire Wire Line
 	6250 1600 6250 1550
@@
 L Device:R_Small R?
 U 1 1 6175B0D8
-P 6000 1700
+P 6000 1800
 AR Path="/6175B0D8" Ref="R?"  Part="1"
 AR Path="/6184F8A1/6175B0D8" Ref="R34"  Part="1"
@@
 AR Path="/61875F91/6175B0D8" Ref="R48"  Part="1"
 AR Path="/61876EF7/6175B0D8" Ref="R55"  Part="1"
-F 0 "R34" H 6059 1746 50  0000 L CNN
-F 1 "DNP" H 6059 1655 50  0000 L CNN
-F 2 "otter:R_0402" H 6000 1700 50  0001 C CNN
-F 3 "~" H 6000 1700 50  0001 C CNN
-	1    6000 1700
+F 0 "R34" H 6059 1846 50  0000 L CNN
+F 1 "DNP" H 6059 1755 50  0000 L CNN
+F 2 "otter:R_0402" H 6000 1800 50  0001 C CNN
+F 3 "~" H 6000 1800 50  0001 C CNN
+	1    6000 1800
 	1    0    0    -1
 $EndComp
@@
 Wire Wire Line
 	6300 1700 6300 2000
-Wire Wire Line
-	6000 1800 6000 2000
-Connection ~ 6000 2000
-Wire Wire Line
-	6000 2000 6300 2000
 $Comp
 L Device:R_Small R?
@@
 P 2000 3950
 AR Path="/617CC90F" Ref="#PWR?"  Part="1"
-AR Path="/6184F8A1/617CC90F" Ref="#PWR?"  Part="1"
-AR Path="/61875035/617CC90F" Ref="#PWR?"  Part="1"
-AR Path="/61875F91/617CC90F" Ref="#PWR?"  Part="1"
-AR Path="/61876EF7/617CC90F" Ref="#PWR?"  Part="1"
-F 0 "#PWR?" H 2000 3800 50  0001 C CNN
+AR Path="/6184F8A1/617CC90F" Ref="#PWR0228"  Part="1"
+AR Path="/61875035/617CC90F" Ref="#PWR0230"  Part="1"
+AR Path="/61875F91/617CC90F" Ref="#PWR0232"  Part="1"
+AR Path="/61876EF7/617CC90F" Ref="#PWR0234"  Part="1"
+F 0 "#PWR0228" H 2000 3800 50  0001 C CNN
 F 1 "+3V3" H 2015 4123 50  0000 C CNN
 F 2 "" H 2000 3950 50  0001 C CNN
@@
 P 2000 4050
 AR Path="/617CC915" Ref="C?"  Part="1"
-AR Path="/6184F8A1/617CC915" Ref="C?"  Part="1"
-AR Path="/61875035/617CC915" Ref="C?"  Part="1"
-AR Path="/61875F91/617CC915" Ref="C?"  Part="1"
-AR Path="/61876EF7/617CC915" Ref="C?"  Part="1"
-F 0 "C?" H 1908 4004 50  0000 R CNN
+AR Path="/6184F8A1/617CC915" Ref="C33"  Part="1"
+AR Path="/61875035/617CC915" Ref="C34"  Part="1"
+AR Path="/61875F91/617CC915" Ref="C35"  Part="1"
+AR Path="/61876EF7/617CC915" Ref="C36"  Part="1"
+F 0 "C33" H 1908 4004 50  0000 R CNN
 F 1 "DNP" H 1908 4095 50  0000 R CNN
 F 2 "otter:C_0402" H 2000 4050 50  0001 C CNN
@@
 P 2000 4150
 AR Path="/617CC91B" Ref="#PWR?"  Part="1"
-AR Path="/6184F8A1/617CC91B" Ref="#PWR?"  Part="1"
-AR Path="/61875035/617CC91B" Ref="#PWR?"  Part="1"
-AR Path="/61875F91/617CC91B" Ref="#PWR?"  Part="1"
-AR Path="/61876EF7/617CC91B" Ref="#PWR?"  Part="1"
-F 0 "#PWR?" H 2000 3900 50  0001 C CNN
+AR Path="/6184F8A1/617CC91B" Ref="#PWR0229"  Part="1"
+AR Path="/61875035/617CC91B" Ref="#PWR0231"  Part="1"
+AR Path="/61875F91/617CC91B" Ref="#PWR0233"  Part="1"
+AR Path="/61876EF7/617CC91B" Ref="#PWR0235"  Part="1"
+F 0 "#PWR0229" H 2000 3900 50  0001 C CNN
 F 1 "GND" H 2005 3977 50  0000 C CNN
 F 2 "" H 2000 4150 60  0000 C CNN
@@
 	1    0    0    -1
 $EndComp
+Wire Wire Line
+	5750 2000 6000 2000
+Wire Wire Line
+	6000 1700 6000 1600
+Wire Wire Line
+	6000 1900 6000 2000
+Connection ~ 6000 2000
+Wire Wire Line
+	6000 2000 6300 2000
 $EndSCHEMATC
